File: mmdvm_hs-hat.sch (KiCad schematic (older format))
At the start: 76 parts, among them P1 I2C, P2 DISPLAY, P3 SMA, P4 STLINK, SW1 DNI, U1 ADF7021, U2 STM32F103C8T6, X1 TCXO, Y1 8MHz

Commit message: Fix ERC warnings, update pin directions on devices.
Connections:
- wire segments 320 -> 327

Commit message: Rotate 180° STLink connector (respect OLED and Nextion orientations). Replace GND pads to VIA (netlist can be safely updated from schematic now). Reroute Service track. Small tweaks to various tracks (WiP). DRC success. Update 3D topview PNG.
Parts:
- C1, C10, C11, C12, C13, C14, C15, C16, C17, C18, C19, C2, C20, C21, C22, C23, C24, C25, C26, C27, C28, C29, C3, C31, C4, C5, C6, C7, C8, C9: footprint Capacitors_SMD:C_0402 -> Capacitor_SMD:C_0402_1005Metric
- C30: footprint Capacitors_Tantalum_SMD:CP_Tantalum_Case-A_EIA-3216-18_Reflow -> Capacitor_Tantalum_SMD:CP_EIA-3216-18_Kemet-A
- D1, D2, D3, D4, D5, D6, D7, D8, D9: footprint LEDs:LED_0402 -> LED_SMD:LED_0402_1005Metric
- L1, L2, L3, L4, L5, L6: footprint Inductors_SMD:L_0402 -> Inductor_SMD:L_0402_1005Metric
- P1, P2, P4: footprint Pin_Headers:Pin_Header_Straight_1x04 -> Connector_PinHeader_2.54mm:PinHeader_1x04_P2.54mm_Vertical
- R1, R10, R11, R12, R13, R14, R15, R16, R17, R18, R19, R2, R3, R4, R5, R6, R7, R8, R9: footprint Resistors_SMD:R_0402 -> Resistor_SMD:R_0402_1005Metric

Commit message: Add I2C OLED on 2x20 connector (should make it optional).
Connections:
- wire segments 327 -> 331
Other:
- note added: "OLED"
Changed lines of the file:
@@
 Wire Wire Line
 	4350 2450 4350 2500
+$Comp
+L power:+3.3V #PWR?
+U 1 1 5B0F1627
+P 3450 1650
+F 0 "#PWR?" H 3450 1500 50  0001 C CNN
+F 1 "+3.3V" H 3450 1790 50  0000 C CNN
+F 2 "" H 3450 1650 50  0000 C CNN
+F 3 "" H 3450 1650 50  0000 C CNN
+	1    3450 1650
+	1    0    0    -1
+$EndComp
+Wire Wire Line
+	2850 1700 3450 1700
+Wire Wire Line
+	3450 1700 3450 1650
+Text GLabel 3350 1900 2    60   Input ~ 0
+SCL
+Text GLabel 3350 2000 2    60   Input ~ 0
+SDA
+Wire Wire Line
+	2850 1900 3350 1900
+Wire Wire Line
+	2850 2000 3350 2000
+Wire Notes Line
+	3250 1450 3950 1450
+Wire Notes Line
+	3950 1450 3950 2250
+Wire Notes Line
+	3950 2250 3250 2250
+Wire Notes Line
+	3250 1450 3250 2250
+Text Notes 3700 2250 0    60   ~ 0
+OLED
 $EndSCHEMATC

Commit message: Make OLED_on_2x20 optionnal, electrically (using 3x0402 unpopulated resistors).
Parts:
- added R20, R21, R22: DNI, Resistor_SMD:R_0402_1005Metric, symbol Device:R
Connections:
- wire segments 331 -> 334
Changed lines of the file:
@@
 	4350 2450 4350 2500
 $Comp
-L power:+3.3V #PWR?
+L power:+3.3V #PWR0102
 U 1 1 5B0F1627
-P 3450 1650
-F 0 "#PWR?" H 3450 1500 50  0001 C CNN
-F 1 "+3.3V" H 3450 1790 50  0000 C CNN
-F 2 "" H 3450 1650 50  0000 C CNN
-F 3 "" H 3450 1650 50  0000 C CNN
-	1    3450 1650
+P 3800 1650
+F 0 "#PWR0102" H 3800 1500 50  0001 C CNN
+F 1 "+3.3V" H 3800 1790 50  0000 C CNN
+F 2 "" H 3800 1650 50  0000 C CNN
+F 3 "" H 3800 1650 50  0000 C CNN
+	1    3800 1650
 	1    0    0    -1
 $EndComp
 Wire Wire Line
-	2850 1700 3450 1700
-Wire Wire Line
-	3450 1700 3450 1650
-Text GLabel 3350 1900 2    60   Input ~ 0
+	3800 1700 3800 1650
+Text GLabel 3650 1900 2    60   Input ~ 0
 SCL
-Text GLabel 3350 2000 2    60   Input ~ 0
+Text GLabel 3650 2000 2    60   Input ~ 0
 SDA
-Wire Wire Line
-	2850 1900 3350 1900
-Wire Wire Line
-	2850 2000 3350 2000
 Wire Notes Line
-	3250 1450 3950 1450
+	3200 1450 3950 1450
 Wire Notes Line
 	3950 1450 3950 2250
 Wire Notes Line
-	3950 2250 3250 2250
+	3950 2250 3200 2250
 Wire Notes Line
-	3250 1450 3250 2250
+	3200 1450 3200 2250
 Text Notes 3700 2250 0    60   ~ 0
 OLED
+$Comp
+L Device:R R20
+U 1 1 5B119166
+P 3450 1700
+F 0 "R20" V 3350 1550 50  0000 C CNN
+F 1 "DNI" V 3450 1700 50  0000 C CNN
+F 2 "Resistor_SMD:R_0402_1005Metric" V 3380 1700 50  0001 C CNN
+F 3 "~" H 3450 1700 50  0001 C CNN
+	1    3450 1700
+	0    1    1    0
+$EndComp
+$Comp
+L Device:R R21
+U 1 1 5B1D838D
+P 3450 1900
+F 0 "R21" V 3350 1750 50  0000 C CNN
+F 1 "DNI" V 3450 1900 50  0000 C CNN
+F 2 "Resistor_SMD:R_0402_1005Metric" V 3380 1900 50  0001 C CNN
+F 3 "~" H 3450 1900 50  0001 C CNN
+	1    3450 1900
+	0    1    1    0
+$EndComp
+$Comp
+L Device:R R22
+U 1 1 5B1D8443
+P 3450 2000
+F 0 "R22" V 3550 1850 50  0000 C CNN
+F 1 "DNI" V 3450 2000 50  0000 C CNN
+F 2 "Resistor_SMD:R_0402_1005Metric" V 3380 2000 50  0001 C CNN
+F 3 "~" H 3450 2000 50  0001 C CNN
+	1    3450 2000
+	0    1    1    0
+$EndComp
+Wire Wire Line
+	3600 1700 3800 1700
+Wire Wire Line
+	3600 1900 3650 1900
+Wire Wire Line
+	3650 2000 3600 2000
+Wire Wire Line
+	3300 2000 2850 2000
+Wire Wire Line
+	3300 1900 2850 1900
+Wire Wire Line
+	3300 1700 2850 1700
 $EndSCHEMATC
